Commit message: change the mass and arm length

File: gym_pybullet_drones/assets/hb.urdf (robot description, URDF)
Before this commit: robot quad, 6 links, 5 joints
Links:
- link base_link: mass 0.5 -> 1.2; geometry collision cylinder length=.15 radius=.22; visual mesh filename=./drone.STL scale=.00075 .00075 .00075

Commit message: change the collision shape to sphere

File: gym_pybullet_drones/assets/hb.urdf (robot description, URDF)
Before this commit: robot quad, 6 links, 5 joints
Links:
- link base_link: geometry collision sphere radius=0.22; visual mesh filename=./drone.STL scale=.00075 .00075 .00075

Commit message: changed the mesh scale of drone

File: gym_pybullet_drones/assets/hb.urdf (robot description, URDF)
Before this commit: robot quad, 6 links, 5 joints
Links:
- link base_link: geometry collision sphere radius=0.22; visual mesh filename=./drone.STL scale=.00095 .00095 .00095
