Commit message: add tree branch to the learning frimwork; unfinished no collision between the drones and branch

File: gym_pybullet_drones/assets/treebranch.urdf (robot description, URDF)
Before this commit: robot tree, 3 links, 2 joints
Links:
- link base_link: geometry collision box size=2.0 2.0 0.5; visual cylinder length=4 radius=0.25

Commit message: change teh branch diameter

File: gym_pybullet_drones/assets/treebranch.urdf (robot description, URDF)
Before this commit: robot tree, 3 links, 2 joints
Links:
- link treebranch_link: geometry collision cylinder length=1.5 radius=0.02; visual cylinder length=1.5 radius=0.02

Commit message: change the branch pos limits

File: gym_pybullet_drones/assets/treebranch.urdf (robot description, URDF)
Before this commit: robot tree, 3 links, 2 joints
Joints:
- joint base_to_virtual_link: limit lower=-0.3 upper=0.3 effort=1000 velocity=0.5 -> lower=-0.0 upper=0.0 effort=1000 velocity=0.5
- joint joint2: limit lower=-1.1 upper=1.3 effort=1000 velocity=0.5 -> lower=-0.0 upper=0.0 effort=1000 velocity=0.5

Commit message: change branch

File: gym_pybullet_drones/assets/treebranch.urdf (robot description, URDF)
Before this commit: robot tree, 3 links, 2 joints
Links:
- link base_link: geometry collision cylinder length=4 radius=0.25; visual cylinder length=4 radius=0.25
- link treebranch_link: geometry collision cylinder length=1.5 radius=0.03; visual cylinder length=1.5 radius=0.03

Commit message: change the branch para

File: gym_pybullet_drones/assets/treebranch.urdf (robot description, URDF)
Before this commit: robot tree, 3 links, 2 joints
Joints:
- joint joint2: limit lower=-0.0 upper=0.0 effort=1000 velocity=0.5 -> lower=-0.3 upper=0.3 effort=1000 velocity=0.5

Commit message: cancel the collision shape of the branch base

File: gym_pybullet_drones/assets/treebranch.urdf (robot description, URDF)
Before this commit: robot tree, 3 links, 2 joints
Links:
- link base_link: geometry visual cylinder length=4 radius=0.25
Joints:
- joint base_to_virtual_link: limit lower=-0.0 upper=0.0 effort=1000 velocity=0.5 -> lower=-0.3 upper=0.3 effort=1000 velocity=0.5

Commit message: changed branch radius

File: gym_pybullet_drones/assets/treebranch.urdf (robot description, URDF)
Before this commit: robot tree, 3 links, 2 joints
Links:
- link treebranch_link: geometry collision cylinder length=1.5 radius=0.01; visual cylinder length=1.5 radius=0.01

Commit message: update for random init tree location

File: gym_pybullet_drones/assets/treebranch.urdf (robot description, URDF)
Before this commit: robot tree, 3 links, 2 joints
Links:
- link base_link: geometry visual cylinder length=2 radius=0.25
Joints:
- joint base_to_virtual_link: origin xyz=0 0 1.75 rpy=0 0 0 -> xyz=0 0 0.6 rpy=0 0 0
